Commit message: Good simulation parameters

File: src/mybot_description/urdf/macros.xacro (robot description, xacro)
@@ -1,6 +1,7 @@
 <?xml version="1.0"?>
 <robot>
-  <!--macro name="cylinder_inertia" params="m r h">
-    <inertia  ixx="${m*(3*r*r+h*h)/12}" ixy = "0" ixz = "0"
+  <macro name="cylinder_inertia" params="m r h">
+    <inertia
+      ixx="${m*(3*r*r+h*h)/12}" ixy = "0" ixz = "0"
       iyy="${m*(3*r*r+h*h)/12}" iyz = "0"
       izz="${m*r*r/2}"
@@ -8,5 +9,6 @@
   </macro>
   <macro name="box_inertia" params="m x y z">
-    <inertia  ixx="${m*(y*y+z*z)/12}" ixy = "0" ixz = "0"
+    <inertia
+      ixx="${m*(y*y+z*z)/12}" ixy = "0" ixz = "0"
       iyy="${m*(x*x+z*z)/12}" iyz = "0"
       izz="${m*(x*x+z*z)/12}"
@@ -14,10 +16,11 @@
   </macro>
   <macro name="sphere_inertia" params="m r">
-    <inertia  ixx="${2*m*r*r/5}" ixy = "0" ixz = "0"
+    <inertia
+      ixx="${2*m*r*r/5}" ixy = "0" ixz = "0"
       iyy="${2*m*r*r/5}" iyz = "0"
       izz="${2*m*r*r/5}"
     />
   </macro>
-  <macro name="wheel" params="lr tY">
+  <!--macro name="wheel" params="lr tY">
     <link name="${lr}_wheel">
       <collision>
@@ -66,4 +69,5 @@
       </actuator>
     </transmission>
-  </macro-->
+  </macro>
+  <-->
 </robot>

File: src/mybot_description/urdf/mybot.xacro (robot description, xacro)
@@ -7,11 +7,7 @@
     <pose>0 0 0 0 0 0</pose>
     <inertial>
-      <mass value="10"/>
+      <mass value="3"/>
       <origin xyz="0 0 0" rpy=" 0 0 0"/>
-      <inertia
-          ixx="0.0" ixy="0" ixz="0"
-          iyy="0.0" iyz="0"
-          izz="0.0"
-      />
+	  <box_inertia m="3" x="0.3" y="0.23" z="0.07"/>
     </inertial>
     <collision name='collision'>
@@ -69,4 +65,7 @@
         <sphere radius="0.0325"/>
       </geometry>
+      <inertial>
+		  <mass value="1"/>
+      </inertial>
     </visual>
     <collision name='caster_collision2'>
@@ -91,4 +90,7 @@
         <sphere radius="0.0325"/>
       </geometry>
+      <inertial>
+		  <mass value="1"/>
+      </inertial>
     </visual>
   </link>
@@ -129,9 +131,5 @@
       <origin xyz="0 0 0" rpy="0 1.5707 1.5707"/>
       <mass value="1"/>
-      <cylinder_inertia m="0.05" r="0.0325" h="0.02"/>
-      <inertia
-        ixx="0.0" ixy="0.0" ixz="0.0"
-        iyy="0.0" iyz="0.0"
-        izz="0.0"/>
+      <cylinder_inertia m="1" r="0.0325" h="0.02"/>
     </inertial>
   </link>
@@ -153,9 +151,5 @@
       <origin xyz="0 0 0" rpy="0 1.5707 1.5707"/>
       <mass value="1"/>
-      <cylinder_inertia m="0.05" r="0.0325" h="0.02"/>
-      <inertia
-        ixx="0.0" ixy="0.0" ixz="0.0"
-        iyy="0.0" iyz="0.0"
-        izz="0.0"/>
+      <cylinder_inertia m="1" r="0.0325" h="0.02"/>
     </inertial>
   </link>
