Commit message: Simulation ready

File: src/mybot_description/urdf/mybot.xacro (robot description, xacro)
@@ -161,5 +161,5 @@
   </joint>
   <joint type="continuous" name="left_wheel_hinge">
-    <origin xyz="0.135 -0.135 -0.035" rpy="0 0 0"/>
+    <origin xyz="0.135 0.135 -0.035" rpy="0 0 0"/>
     <child link="left_wheel"/>
     <parent link="chassis"/>
@@ -169,5 +169,5 @@
   </joint>
   <joint type="continuous" name="right_wheel_hinge">
-    <origin xyz="0.135 0.135 -0.035" rpy="0 0 0"/>
+    <origin xyz="0.135 -0.135 -0.035" rpy="0 0 0"/>
     <child link="right_wheel"/>
     <parent link="chassis"/>
@@ -214,6 +214,5 @@
       </inertial>
     </link>
-    <!-- The fixed joints & links below are usually published by static_transformers launched by the OpenNi launch
-         files. However, for Gazebo simulation we need them, so we add them here.
+    <!-- The fixed joints & links below are usually published by static_transformers launched by the OpenNi launch files. However, for Gazebo simulation we need them, so we add them here.
          (Hence, don't publish them additionally!) -->
 	<joint name="camera_depth_joint" type="fixed">
